Commit message: Simulation finally works     Solved tons of issues, including:     - Fixed the issue with the robot not moving in simulation.     - Fixed the issue with the robot not being able to see the goal.     - Reestructured the code to make it more readable and maintainable.     - Added a new launch file to run the simulation with the robot.

File: src/blackpearls_nav2_puzzlebot/urdf/puzzlebot.urdf (robot description, URDF)
Before this commit: robot Puzzlebot_Jetson_Lidar_Ed., 5 links, 4 joints
Links:
- link base_link: geometry visual mesh filename=package://blackpearls_nav2_puzzlebot/meshes/Puzzlebot_Jetso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
- link caster_wheel_link: geometry visual mesh filename=package://blackpearls_nav2_puzzlebot/meshes/Puzzlebot_Caste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
- link wheel_left: geometry visual mesh filename=package://blackpearls_nav2_puzzlebot/meshes/Puzzlebot_Wheel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
- link wheel_right: geometry visual mesh filename=package://blackpearls_nav2_puzzlebot/meshes/Puzzlebot_Wheel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
