Commit message: Spawn Puzzlebot in gazebo  garden.

File: blackpearls_nav2_puzzlebot/urdf/puzzlebot.urdf (robot description, URDF)
Before this commit: robot Puzzlebot_Jetson_Lidar_Ed., 5 links, 4 joints
Links:
- link base_footprint: mass None -> 2.0
- link base_link: mass None -> 2.0
- link caster_wheel_link: mass None -> 2.0
- link wheel_left: mass None -> 2.0
- link wheel_right: mass None -> 2.0

Commit message: Actividad M3.4: Simulación proyecto final corrección 3

File: blackpearls_nav2_puzzlebot/urdf/puzzlebot.urdf (robot description, URDF)
Before this commit: robot Puzzlebot_Jetson_Lidar_Ed., 5 links, 4 joints
Links:
- removed link caster_wheel_link
- removed link wheel_left
- removed link wheel_right
- added link caster_link, mass 2.0; visual mesh filename=package://blackpearls_nav2_puzzlebot/meshes/Puzzlebot_Caste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
- added link wheel_l_link, mass 2.0; visual mesh filename=package://blackpearls_nav2_puzzlebot/meshes/Puzzlebot_Wheel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
- added link wheel_r_link, mass 2.0; visual mesh filename=package://blackpearls_nav2_puzzlebot/meshes/Puzzlebot_Wheel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
Joints:
- removed joint caster_wheel_joint
- removed joint wheel_left_joint
- removed joint wheel_right_joint
- added joint caster_joint: type fixed, parent base_link, child caster_link, origin xyz=-0.095 0 -0.03 rpy=0 0 0
- added joint wheel_l_joint: type continuous, parent base_link, child wheel_l_link, origin xyz=0.052 0.095 -0.0025 rpy=0 0 0, axis 0 1 0 
- added joint wheel_r_joint: type continuous, parent base_link, child wheel_r_link, origin xyz=0.052 -0.095 -0.0025 rpy=0 0 0, axis 0 1 0 

Commit message: Added the final details

File: blackpearls_nav2_puzzlebot/urdf/puzzlebot.urdf (robot description, URDF)
Before this commit: robot Puzzlebot_Jetson_Lidar_Ed., 5 links, 4 joints
Links:
- link base_link: geometry visual mesh filename=package://blackpearls_nav2_puzzlebot/meshes/meshes_old/MCR2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
